File: PSLab KiCAD/IO.sch (KiCad schematic (older format))
At the start: 69 parts, among them P1 CONN_01X08, P11 47K, Q1 3906, U10 TL082, U11 6S21, U12 6S21, U13 TL082, U16 TL082, U7 LM324, U8 TL082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

Commit message: Edited R11 value and changed zener voltages
Parts:
- U9: symbol MCP4728 -> MCP4728-RESCUE-PSLab
Changed lines of the file:
@@
 $EndComp
 $Comp
-L MCP4728 U9
+L MCP4728-RESCUE-PSLab U9
 U 1 1 555FFB01
 P 1650 1800
