File: PSLab KiCAD/PSLab.sch (KiCad schematic (older format))
At the start: 71 parts, among them CON1 USB-MINI-B, P10 Analog, P12 5V, P13 MCLR, P2 PROG, P3 DIO, P4 V+/V-, P5 sen-cap, P6 I2C, P7 NRF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

Commit message: Edited R11 value and changed zener voltages
Parts:
- added Battery: 12V, symbol Battery
- added D?: 5V, symbol ZENERsmall-RESCUE-proto1
- added R1: 100, symbol R
- D3, D4: symbol LED -> LED-RESCUE-PSLab
- U6: symbol LM1117-3.3 -> LM1117-3.3-RESCUE-PSLab
Connections:
- net labels added: Output
- wire segments 215 -> 223
