File: PSLab KiCAD v2/PSLab.kicad_pcb (KiCad board)
At the start: 4 copper layers, 60 x 75 mm, 144 parts, among them CON1 USB-MINI-B, P1 CONN_01X08, P10 Analog, P11 47K, P12 5V, P13 MCLR, P2 PROG, P3 DIO, P4 V+/V-, P5 sen-cap, P6 I2C, P7 NRF, P8 CONN_02X10, P9 Tx-Rx, Q1 3906, Q2 BT5551, U1 MCP2200, U10 TL082, U11 6S21, U12 6S21, U13 TL082, U14 WS2182, U15 ESP8266, U16 TL082, U17 FOX924B, U2 74HC126, U3 PIC24EP64GP204, U4 TC1240A, U5 7660, U6 LM1117-3.3, U7 LM324, U8 TL082, U9 MCP4728

Commit message: Fix #16 : PCB Layout for Voltage Regulator
Parts:
- added Q3: MMBT3906, TO_SOT_Packages_SMD:SOT-23, F.Cu at (134.4, 93.5)
- Q2: value BT5551 -> MMBT3904
- R11, R5: value 200 -> 1K
Connections:
- net VUSB renamed Net-(CON1-Pad1)
- D1 pad 2: VR+ -> Net-(D1-Pad2)
- D2 pad 1: VR- -> Net-(D2-Pad1)
- Q2 pad 1: Net-(C3-Pad1) -> Net-(D1-Pad2)
- Q2 pad 2: GND -> VR+
- Q2 pad 3: Net-(L2-Pad1) -> V+
- R11 pad 1: VR- -> V-
- R11 pad 2: V- -> Net-(D2-Pad1)
- R5 pad 1: VR+ -> Net-(D1-Pad2)
Routing:
- net Net-(D2-Pad1): track 0.00 -> 37.5 mm, vias 0 -> 2
- net V-: track 92.0 -> 122.8 mm, vias 3 -> 6
- net VR-: track 75.0 -> 54.9 mm, vias 4 -> 1
- net Net-(D1-Pad2): track 0.00 -> 9.24 mm
- net Net-(C3-Pad1): track 10.2 -> 3.49 mm
- net Net-(L2-Pad1): track 5.69 -> 2.31 mm
- net V+: track 74.1 -> 77.5 mm
- net VR+: track 75.0 -> 72.5 mm
