File: PSLab KiCAD v3/IO.sch (KiCad schematic (older format))
At the start: 68 parts, among them P1 CONN_01X08, Q1 3906, U10 TL082, U11 6S21, U12 6S21, U13 TL082, U16 TL082, U7 LM324, U8 TL082, U9 MCP4728

Commit message: Added Gerber files
Parts:
- removed Q1: 3906, TO_SOT_Packages_SMD:SOT-23, symbol 3906
- added Q1: MMBT3906, TO_SOT_Packages_SMD:SOT-23, symbol MMBT3906
Connections:
- net PCS: now also Q1.3 (C)
- net at U7.8: now also Q1.1 (B)
- net at R36.2, U7.9 (-): now also Q1.2 (E)
Changed lines of the file:
@@
 Text GLabel 2000 1950 2    40   Input ~ 0
 PVS3
-$Comp
-L 3906 Q1
-U 1 1 5560A90C
-P 2050 2875
-F 0 "Q1" H 2250 2775 50  0000 C CNN
-F 1 "3906" H 2325 2900 50  0000 C CNN
-F 2 "TO_SOT_Packages_SMD:SOT-23" H 2050 2875 60  0001 C CNN
-F 3 "" H 2050 2875 60  0000 C CNN
-	1    2050 2875
-	1    0    0    -1
-$EndComp
 Text GLabel 2325 2575 2    40   Input ~ 0
 PCS
@@
 Wire Wire Line
 	1240 4765 1295 4765
+$Comp
+L MMBT3906 Q1
+U 1 1 5A3360AB
+P 2050 2875
+F 0 "Q1" H 2240 2965 50  0000 L CNN
+F 1 "MMBT3906" H 2245 2790 50  0000 L CNN
+F 2 "TO_SOT_Packages_SMD:SOT-23" H 2250 2800 50  0001 L CIN
+F 3 "" H 2050 2875 50  0001 L CNN
+	1    2050 2875
+	1    0    0    -1
+$EndComp
 $EndSCHEMATC
