File: PSLab KiCAD v4/PSLab.sch (KiCad schematic (older format))
At the start: 79 parts, among them CON1 USB-MINI-B, J1 Programmer, J10 GND, J11 Vbus, J12 Sensors, J13 D+, J14 D-, J16 I2C-2, J2 SQRs, J3 LA, J4 OSC_Pins, J6 I2C-1, J7 IDs, J8 Conn_01x07, P7 NRF, Q2 MMBT3904, Q3 MMBT3906, U1 MCP2200, U15 ESP8266, U2 74HC126, U3 PIC24EP256GP204, U4 TC1240A, U5 7660, U6 LM1117-3.3, X1 12MHz, Y1 12MHz

Commit message: Refined BOM Sheet
Parts:
- removed C15, C21: 10u, Capacitors_SMD:C_0603, symbol CAPAPOL
- removed J12: Sensors, Pin_Headers:Pin_Header_Straight_2x03_Pitch2.54mm, symbol Conn_02x03_Odd_Even
- removed J2: SQRs, Pin_Headers:Pin_Header_Straight_1x08_Pitch2.54mm, symbol Conn_01x08
- removed J4: OSC_Pins, Pin_Headers:Pin_Header_Straight_2x07_Pitch2.54mm, symbol Conn_02x07_Odd_Even
- removed J7: IDs, Pin_Headers:Pin_Header_Straight_2x04_Pitch2.54mm, symbol Conn_02x04_Odd_Even
- added C15, C21: 10u, Capacitors_SMD:C_0603, symbol C-RESCUE-proto1
- added J2: DoublePins, Pin_Headers:Pin_Header_Straight_2x14_Pitch2.54mm, symbol Conn_02x14_Odd_Even
- C10, C8: value 33pF -> 33p
- MH1, MH2, MH3, MH4: footprint Mounting_Holes:MountingHole_2.2mm_M2_ISO14580_Pad -> Mounting_Holes:MountingHole_3.2mm_M3_DIN965_Pad
- R48: value 5k1 -> 5K1
Connections:
- net ACH1: now also J2.19 (Pin_19)
- net AN8: now also J2.1 (Pin_1)
- net CAP: now also J2.5 (Pin_5)
- net CH1: now also J2.17 (Pin_17)
- net CH2: now also J2.15 (Pin_15)
- net CH3: now also J2.13 (Pin_13)
- net CH3.GAIN: now also J2.11 (Pin_11)
- net FCin: now also J2.7 (Pin_7)
- net GND: now also C15.1, C21.1, J2.10 (Pin_10), J2.12 (Pin_12), J2.14 (Pin_14), J2.16 (Pin_16), J2.18 (Pin_18), J2.2 (Pin_2), J2.20 (Pin_20), J2.22 (Pin_22), J2.24 (Pin_24), J2.26 (Pin_26), J2.28 (Pin_28), J2.4 (Pin_4), J2.6 (Pin_6), J2.8 (Pin_8)
- net MIC: now also J2.9 (Pin_9)
- net SEN: now also J2.3 (Pin_3)
- net Vdd: now also C15.2
- net IDB: now reaches J3.3 (Pin_3), R7.1
- net IDB: now also J2.23 (Pin_23)
- net IDA: now reaches J3.4 (Pin_4), R6.1
- net IDA: now also J2.21 (Pin_21)
- net at U3.7 (Vcap): now also C21.2
- net IDC: now reaches J3.2 (Pin_2), R8.1
- net IDC: now also J2.25 (Pin_25)
- net IDD: now reaches J3.1 (Pin_1), R9.1
- net IDD: now also J2.27 (Pin_27)
Other:
- note added: "Logic Analyzer"
- moved on the sheet: J3

Commit message: Added FOSSASIA Logo and updated BoM
Parts:
- C3, C43: symbol C -> C-RESCUE-proto1
- R48: symbol R -> R-RESCUE-proto1
Connections:
- net IDA: now also J2.27 (Pin_27); no longer J2.21 (Pin_21)
- net IDB: now also J2.25 (Pin_25); no longer J2.23 (Pin_23)
- net IDC: now also J2.23 (Pin_23); no longer J2.25 (Pin_25)
- net IDD: now also J2.21 (Pin_21); no longer J2.27 (Pin_27)
Other:
- moved on the sheet: R48
Changed lines of the file:
@@
 Text GLabel 3325 3875 0    40   Output ~ 0
 SQ4
-$Comp
-L GND-RESCUE-proto1 #PWR041
-U 1 1 5564F446
-P 8350 1225
-F 0 "#PWR041" H 8350 1225 30  0001 C CNN
-F 1 "GND" H 8350 1155 30  0001 C CNN
-F 2 "" H 8350 1225 60  0000 C CNN
-F 3 "" H 8350 1225 60  0000 C CNN
-	1    8350 1225
-	0    1    1    0
-$EndComp
-$Comp
-L C-RESCUE-proto1 C2
-U 1 1 5564F04A
-P 8550 1225
-F 0 "C2" H 8550 1325 40  0000 L CNN
-F 1 "0.1u" H 8556 1140 40  0000 L CNN
-F 2 "Capacitors_SMD:C_0603" H 8588 1075 30  0001 C CNN
-F 3 "" H 8550 1225 60  0000 C CNN
-	1    8550 1225
-	0    -1   -1   0
-$EndComp
 Text GLabel 6085 6765 0    40   Input ~ 0
 CH3
@@
 ACH1
 $Comp
-L PWR_FLAG #FLG042
+L PWR_FLAG #FLG041
 U 1 1 55EA2B09
 P 3060 5890
-F 0 "#FLG042" H 3060 5985 30  0001 C CNN
+F 0 "#FLG041" H 3060 5985 30  0001 C CNN
 F 1 "PWR_FLAG" H 3225 5970 30  0000 C CNN
 F 2 "" H 3060 5890 60  0000 C CNN
@@
 $EndComp
 $Comp
-L GND-RESCUE-proto1 #PWR043
+L GND-RESCUE-proto1 #PWR042
 U 1 1 5660E9DB
 P 9270 5520
-F 0 "#PWR043" H 9270 5520 30  0001 C CNN
+F 0 "#PWR042" H 9270 5520 30  0001 C CNN
 F 1 "GND" H 9270 5450 30  0001 C CNN
 F 2 "" H 9270 5520 60  0000 C CNN
@@
 $EndComp
 $Comp
-L GND-RESCUE-proto1 #PWR044
+L GND-RESCUE-proto1 #PWR043
 U 1 1 566130A1
 P 9270 5940
-F 0 "#PWR044" H 9270 5940 30  0001 C CNN
+F 0 "#PWR043" H 9270 5940 30  0001 C CNN
 F 1 "GND" H 9270 5870 30  0001 C CNN
 F 2 "" H 9270 5940 60  0000 C CNN
@@
 Mounting Holes
 $Comp
-L GND-RESCUE-proto1 #PWR045
+L GND-RESCUE-proto1 #PWR044
 U 1 1 556DA7E3
 P 1860 1140
-F 0 "#PWR045" H 1860 1140 30  0001 C CNN
+F 0 "#PWR044" H 1860 1140 30  0001 C CNN
 F 1 "GND" H 1860 1070 30  0001 C CNN
 F 2 "" H 1860 1140 60  0000 C CNN
@@
 $EndComp
 $Comp
-L GND-RESCUE-proto1 #PWR046
+L GND-RESCUE-proto1 #PWR045
 U 1 1 5A56D115
 P 5370 7280
-F 0 "#PWR046" H 5370 7280 30  0001 C CNN
+F 0 "#PWR045" H 5370 7280 30  0001 C CNN
 F 1 "GND" H 5370 7210 30  0001 C CNN
 F 2 "" H 5370 7280 60  0000 C CNN
@@
 $EndComp
 $Comp
-L GND-RESCUE-proto1 #PWR047
+L GND-RESCUE-proto1 #PWR046
 U 1 1 5A56FD6E
 P 10165 5835
-F 0 "#PWR047" H 10165 5835 30  0001 C CNN
+F 0 "#PWR046" H 10165 5835 30  0001 C CNN
 F 1 "GND" H 10165 5765 30  0001 C CNN
 F 2 "" H 10165 5835 60  0000 C CNN
@@
 $EndComp
 $Comp
-L GND-RESCUE-proto1 #PWR048
+L GND-RESCUE-proto1 #PWR047
 U 1 1 5A5701EC
 P 10470 5835
-F 0 "#PWR048" H 10470 5835 30  0001 C CNN
+F 0 "#PWR047" H 10470 5835 30  0001 C CNN
 F 1 "GND" H 10470 5765 30  0001 C CNN
 F 2 "" H 10470 5835 60  0000 C CNN
@@
 $EndComp
 $Comp
-L GND-RESCUE-proto1 #PWR049
+L GND-RESCUE-proto1 #PWR048
 U 1 1 5A66B8E0
 P 2285 1925
-F 0 "#PWR049" H 2285 1925 30  0001 C CNN
+F 0 "#PWR048" H 2285 1925 30  0001 C CNN
 F 1 "GND" H 2285 1855 30  0001 C CNN
 F 2 "" H 2285 1925 60  0000 C CNN
@@
 $EndComp
 $Comp
-L R R48
+L R-RESCUE-proto1 R48
 U 1 1 5A6CD97F
-P 3265 2600
-F 0 "R48" V 3345 2600 50  0000 C CNN
-F 1 "5K1" V 3265 2600 50  0000 C CNN
-F 2 "Resistors_SMD:R_0603" V 3195 2600 50  0001 C CNN
-F 3 "" H 3265 2600 50  0001 C CNN
-	1    3265 2600
+P 3365 2600
+F 0 "R48" V 3445 2600 50  0000 C CNN
+F 1 "5K1" V 3365 2600 50  0000 C CNN
+F 2 "Resistors_SMD:R_0603" V 3295 2600 50  0001 C CNN
+F 3 "" H 3365 2600 50  0001 C CNN
+	1    3365 2600
 	0    1    1    0
 $EndComp
-Text Label 3470 2600 0    60   ~ 0
+Text Label 3615 2600 0    60   ~ 0
 Vdd
 $Comp
@@
 $EndComp
 $Comp
-L C C3
+L C-RESCUE-proto1 C3
 U 1 1 5A6D2A55
-P 1425 2365
-F 0 "C3" H 1450 2465 50  0000 L CNN
-F 1 "33p" H 1450 2265 50  0000 L CNN
-F 2 "Capacitors_SMD:C_0603" H 1463 2215 50  0001 C CNN
-F 3 "" H 1425 2365 50  0001 C CNN
-	1    1425 2365
-	1    0    0    -1
-$EndComp
-$Comp
-L C C43
+P 1425 2380
+F 0 "C3" H 1450 2480 50  0000 L CNN
+F 1 "33p" H 1450 2280 50  0000 L CNN
+F 2 "Capacitors_SMD:C_0603" H 1463 2230 50  0001 C CNN
+F 3 "" H 1425 2380 50  0001 C CNN
+	1    1425 2380
+	1    0    0    -1
+$EndComp
+$Comp
+L C-RESCUE-proto1 C43
 U 1 1 5A6D2B78
-P 1965 2370
-F 0 "C43" H 1990 2470 50  0000 L CNN
-F 1 "33p" H 1990 2270 50  0000 L CNN
-F 2 "Capacitors_SMD:C_0603" H 2003 2220 50  0001 C CNN
-F 3 "" H 1965 2370 50  0001 C CNN
-	1    1965 2370
-	1    0    0    -1
-$EndComp
-$Comp
-L GND-RESCUE-proto1 #PWR050
+P 1965 2365
+F 0 "C43" H 1990 2465 50  0000 L CNN
+F 1 "33p" H 1990 2265 50  0000 L CNN
+F 2 "Capacitors_SMD:C_0603" H 2003 2215 50  0001 C CNN
+F 3 "" H 1965 2365 50  0001 C CNN
+	1    1965 2365
+	1    0    0    -1
+$EndComp
+$Comp
+L GND-RESCUE-proto1 #PWR049
 U 1 1 5A6D3C13
 P 1695 2665
-F 0 "#PWR050" H 1695 2665 30  0001 C CNN
+F 0 "#PWR049" H 1695 2665 30  0001 C CNN
 F 1 "GND" H 1695 2595 30  0001 C CNN
 F 2 "" H 1695 2665 60  0000 C CNN
@@
 $EndComp
 $Comp
-L GND-RESCUE-proto1 #PWR051
+L GND-RESCUE-proto1 #PWR050
 U 1 1 5A6F58C4
 P 10775 5835
-F 0 "#PWR051" H 10775 5835 30  0001 C CNN
+F 0 "#PWR050" H 10775 5835 30  0001 C CNN
 F 1 "GND" H 10775 5765 30  0001 C CNN
 F 2 "" H 10775 5835 60  0000 C CNN
@@
 $EndComp
 $Comp
-L GND-RESCUE-proto1 #PWR052
+L GND-RESCUE-proto1 #PWR051
 U 1 1 5A6F5AA9
 P 9855 5840
-F 0 "#PWR052" H 9855 5840 30  0001 C CNN
+F 0 "#PWR051" H 9855 5840 30  0001 C CNN
 F 1 "GND" H 9855 5770 30  0001 C CNN
 F 2 "" H 9855 5840 60  0000 C CNN
@@
 $EndComp
 $Comp
-L GND-RESCUE-proto1 #PWR053
+L GND-RESCUE-proto1 #PWR052
 U 1 1 5AD48170
 P 4195 7080
-F 0 "#PWR053" H 4195 7080 30  0001 C CNN
+F 0 "#PWR052" H 4195 7080 30  0001 C CNN
 F 1 "GND" H 4195 7010 30  0001 C CNN
 F 2 "" H 4195 7080 60  0000 C CNN
@@
 $EndComp
 $Comp
-L GND-RESCUE-proto1 #PWR054
+L GND-RESCUE-proto1 #PWR053
 U 1 1 5AD4BD5F
 P 6875 1895
-F 0 "#PWR054" H 6875 1895 30  0001 C CNN
+F 0 "#PWR053" H 6875 1895 30  0001 C CNN
 F 1 "GND" H 6875 1825 30  0001 C CNN
 F 2 "" H 6875 1895 60  0000 C CNN
@@
 Text GLabel 1135 5135 2    40   Input ~ 0
 IDD
+Text GLabel 6085 7165 0    40   Input ~ 0
+IDD
+Text GLabel 6085 7265 0    40   Input ~ 0
+IDC
+Text GLabel 6085 7365 0    40   Input ~ 0
+IDB
 Text GLabel 6085 7465 0    40   Input ~ 0
-IDD
-Text GLabel 6085 7365 0    40   Input ~ 0
-IDC
-Text GLabel 6085 7265 0    40   Input ~ 0
-IDB
-Text GLabel 6085 7165 0    40   Input ~ 0
 IDA
 Text GLabel 6570 4525 2    40   Input ~ 0
@@
 	3050 2600 3115 2600
 Wire Wire Line
-	3415 2600 3630 2600
-Wire Wire Line
 	1865 2155 2050 2155
 Wire Wire Line
-	1965 2155 1965 2220
-Wire Wire Line
 	1380 2155 1565 2155
 Wire Wire Line
-	1425 2155 1425 2215
-Wire Wire Line
-	1425 2515 1425 2595
-Wire Wire Line
 	1425 2595 1965 2595
-Wire Wire Line
-	1965 2595 1965 2520
 Wire Wire Line
 	1695 2665 1695 2595
 Connection ~ 1695 2595
-Connection ~ 1965 2155
-Connection ~ 1425 2155
 Wire Wire Line
 	2850 2480 2850 2450
@@
 	-1   0    0    1
 $EndComp
+Wire Wire Line
+	1425 2580 1425 2595
+Wire Wire Line
+	1425 2180 1425 2155
+Connection ~ 1425 2155
+Wire Wire Line
+	1965 2595 1965 2565
+Wire Wire Line
+	1965 2165 1965 2155
+Connection ~ 1965 2155
+$Comp
+L GND-RESCUE-proto1 #PWR041
+U 1 1 5564F446
+P 8350 1225
+F 0 "#PWR041" H 8350 1225 30  0001 C CNN
+F 1 "GND" H 8350 1155 30  0001 C CNN
+F 2 "" H 8350 1225 60  0000 C CNN
+F 3 "" H 8350 1225 60  0000 C CNN
+	1    8350 1225
+	0    1    1    0
+$EndComp
+$Comp
+L C-RESCUE-proto1 C2
+U 1 1 5564F04A
+P 8550 1225
+F 0 "C2" H 8550 1325 40  0000 L CNN
+F 1 "0.1u" H 8556 1140 40  0000 L CNN
+F 2 "Capacitors_SMD:C_0603" H 8588 1075 30  0001 C CNN
+F 3 "" H 8550 1225 60  0000 C CNN
+	1    8550 1225
+	0    -1   -1   0
+$EndComp
 $EndSCHEMATC
