File: PSLab KiCAD v4/IO.sch (KiCad schematic (older format))
At the start: 72 parts, among them J15 PCs, J4 Outputs, J9 PVs, Q1 MMBT3906, U10 TL082, U11 6S21, U12 6S21, U13 TL082, U16 TL082, U7 LM324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

Commit message: Added FOSSASIA Logo and updated BoM
Parts:
- removed RV1: POT, Potentiometers:Potentiometer_Alps_RK09K_Vertical, symbol POT
- added R50: 200K, Resistors_SMD:R_0603, symbol R-RESCUE-proto1
Connections:
- net GND: now also R50.2
- net at C6.2: now also R43.1, R50.1
Other:
- moved on the sheet: C6
