File: PSLab KiCAD v4/IO.sch (KiCad schematic (older format))
At the start: 72 parts, among them J15 PCs, J4 Outputs, J9 PVs, Q1 MMBT3906, U10 TL082, U11 6S21, U12 6S21, U13 TL082, U16 TL082, U7 LM324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

Commit message: NRF replaced with Bluetooth
Parts:
- removed J15: PCs, Pin_Headers:Pin_Header_Straight_1x02_Pitch2.54mm, symbol Conn_01x02
- removed J9: PVs, Pin_Headers:Pin_Header_Straight_1x06_Pitch2.54mm, symbol Conn_01x06
- added J8: Power Pins, Pin_Headers:Pin_Header_Straight_1x08_Pitch2.54mm, symbol Conn_01x08
Connections:
- net GND: now also J8.2 (Pin_2), J8.4 (Pin_4), J8.6 (Pin_6), J8.8 (Pin_8)
- net PCS: now also J8.7 (Pin_7)
- net PVS1: now also J8.1 (Pin_1)
- net PVS2: now also J8.3 (Pin_3)
- net PVS3: now also J8.5 (Pin_5)
Other:
- moved on the sheet: TP1, TP2
