File: schematics/Logos.sch (KiCad schematic (older format))
At the start: 10 parts

Commit message: PSLab V6 (#93)
* board: component placement in v6

components: added footprints for regulator and SDcard

routes: voltage regulator, SD card, SPI

components: added tact switch and routes

* board: switch to latest KiCAD version

route: fix switch routes

fix: DRC Issues fixed

docs: added new schematics PDF

docs: updated BoM for v6 PSLab

* feat: 3D models with new KiCAD version

route: VDD missing routes being fixed

route: UART routes

route: complete

3D footprints and optimization

* route: optimization

route: finalized

layout: generated gerber, svg and dxf files for production

* docs: updated BoM

* update: added spacing with more test points

* docs: verrification of BoM

* docs: updated POS files
Parts:
- S1, S10, S2, S3, S4, S5, S6, S7, S8, S9: symbol Logos -> PSLab:Logos
Changed lines of the file:
@@
-EESchema Schematic File Version 2
-LIBS:power
-LIBS:device
-LIBS:transistors
-LIBS:linear
-LIBS:regul
-LIBS:74xx
-LIBS:cmos4000
-LIBS:adc-dac
-LIBS:memory
-LIBS:xilinx
-LIBS:microcontrollers
-LIBS:dsp
-LIBS:microchip
-LIBS:analog_switches
-LIBS:motorola
-LIBS:texas
-LIBS:intel
-LIBS:audio
-LIBS:interface
-LIBS:digital-audio
-LIBS:philips
-LIBS:display
-LIBS:cypress
-LIBS:siliconi
-LIBS:opto
-LIBS:atmel
-LIBS:contrib
-LIBS:valves
-LIBS:conn
-LIBS:PSLab
+EESchema Schematic File Version 4
 LIBS:PSLab-cache
-EELAYER 25 0
+EELAYER 26 0
 EELAYER END
 $Descr A4 11693 8268
 encoding utf-8
-Sheet 3 3
+Sheet 3 5
 Title "PSLab"
 Date "2018-12-29"
@@
 $EndDescr
 $Comp
-L Logos S1
+L PSLab:Logos S1
 U 1 1 5C27C643
 P 4560 2845
@@
 $EndComp
 $Comp
-L Logos S3
+L PSLab:Logos S3
 U 1 1 5C27C831
 P 5460 2845
@@
 $EndComp
 $Comp
-L Logos S6
+L PSLab:Logos S6
 U 1 1 5C27C867
 P 6460 2845
@@
 $EndComp
 $Comp
-L Logos S8
+L PSLab:Logos S8
 U 1 1 5C27C8A4
 P 7410 2845
@@
 $EndComp
 $Comp
-L Logos S2
+L PSLab:Logos S2
 U 1 1 5C27C95E
 P 4560 3545
@@
 $EndComp
 $Comp
-L Logos S4
+L PSLab:Logos S4
 U 1 1 5C27C964
 P 5460 3545
@@
 $EndComp
 $Comp
-L Logos S7
+L PSLab:Logos S7
 U 1 1 5C27C96A
 P 6460 3545
@@
 $EndComp
 $Comp
-L Logos S9
+L PSLab:Logos S9
 U 1 1 5C27C970
 P 7410 3545
@@
 $EndComp
 $Comp
-L Logos S5
+L PSLab:Logos S5
 U 1 1 5C27C986
 P 5560 4195
@@
 $EndComp
 $Comp
-L Logos S10
+L PSLab:Logos S10
 U 1 1 5C27CF8C
 P 6460 4195

Commit message: route: clean ups and optimization
Parts:
- removed S4: App_Barcode, Custom_Components:Barcode, symbol PSLab:Logos
Other:
- moved on the sheet: S2, S7, S9
Changed lines of the file:
@@
 L PSLab:Logos S2
 U 1 1 5C27C95E
-P 4560 3545
-F 0 "S2" H 4560 3425 60  0000 C CNN
-F 1 "PSLab_Logo" H 4560 3665 60  0000 C CNN
-F 2 "Custom_Components:PSLab_Logo" H 4560 3545 60  0001 C CNN
-F 3 "" H 4560 3545 60  0001 C CNN
-	1    4560 3545
-	1    0    0    -1
-$EndComp
-$Comp
-L PSLab:Logos S4
-U 1 1 5C27C964
-P 5460 3545
-F 0 "S4" H 5460 3425 60  0000 C CNN
-F 1 "App_Barcode" H 5460 3665 60  0000 C CNN
-F 2 "Custom_Components:Barcode" H 5460 3545 60  0001 C CNN
-F 3 "" H 5460 3545 60  0001 C CNN
-	1    5460 3545
+P 5070 3515
+F 0 "S2" H 5070 3395 60  0000 C CNN
+F 1 "PSLab_Logo" H 5070 3635 60  0000 C CNN
+F 2 "Custom_Components:PSLab_Logo" H 5070 3515 60  0001 C CNN
+F 3 "" H 5070 3515 60  0001 C CNN
+	1    5070 3515
 	1    0    0    -1
 $EndComp
@@
 L PSLab:Logos S7
 U 1 1 5C27C96A
-P 6460 3545
-F 0 "S7" H 6460 3425 60  0000 C CNN
-F 1 "PSL_Logo" H 6460 3665 60  0000 C CNN
-F 2 "Custom_Components:PSL_Logo" H 6460 3545 60  0001 C CNN
-F 3 "" H 6460 3545 60  0001 C CNN
-	1    6460 3545
+P 5965 3520
+F 0 "S7" H 5965 3400 60  0000 C CNN
+F 1 "PSL_Logo" H 5965 3640 60  0000 C CNN
+F 2 "Custom_Components:PSL_Logo" H 5965 3520 60  0001 C CNN
+F 3 "" H 5965 3520 60  0001 C CNN
+	1    5965 3520
 	1    0    0    -1
 $EndComp
@@
 L PSLab:Logos S9
 U 1 1 5C27C970
-P 7410 3545
-F 0 "S9" H 7410 3425 60  0000 C CNN
-F 1 "QR_Code" H 7410 3665 60  0000 C CNN
-F 2 "Custom_Components:Website_QR" H 7410 3545 60  0001 C CNN
-F 3 "" H 7410 3545 60  0001 C CNN
-	1    7410 3545
+P 6915 3520
+F 0 "S9" H 6915 3400 60  0000 C CNN
+F 1 "QR_Code" H 6915 3640 60  0000 C CNN
+F 2 "Custom_Components:Website_QR" H 6915 3520 60  0001 C CNN
+F 3 "" H 6915 3520 60  0001 C CNN
+	1    6915 3520
 	1    0    0    -1
 $EndComp

Commit message: docs: updated output files
Parts:
- added S4: PSLabDotIO_B, Custom_Components:PSLabDotIO4000, symbol PSLab:Logos
- S1: footprint Symbols:OSHW-Logo2_7.3x6mm_SilkScreen -> Symbols:OSHW-Logo_5.7x6mm_SilkScreen
- S2: footprint Custom_Components:PSLab_Logo -> Custom_Components:PSLabDotIO
Other:
- moved on the sheet: S10, S5
Changed lines of the file:
@@
 F 0 "S1" H 4560 2725 60  0000 C CNN
 F 1 "OpenHardware" H 4560 2965 60  0000 C CNN
-F 2 "Symbols:OSHW-Logo2_7.3x6mm_SilkScreen" H 4560 2845 60  0001 C CNN
+F 2 "Symbols:OSHW-Logo_5.7x6mm_SilkScreen" H 4560 2845 60  0001 C CNN
 F 3 "" H 4560 2845 60  0001 C CNN
 	1    4560 2845
@@
 F 0 "S2" H 5070 3395 60  0000 C CNN
 F 1 "PSLab_Logo" H 5070 3635 60  0000 C CNN
-F 2 "Custom_Components:PSLab_Logo" H 5070 3515 60  0001 C CNN
+F 2 "Custom_Components:PSLabDotIO" H 5070 3515 60  0001 C CNN
 F 3 "" H 5070 3515 60  0001 C CNN
 	1    5070 3515
@@
 L PSLab:Logos S5
 U 1 1 5C27C986
-P 5560 4195
-F 0 "S5" H 5560 4075 60  0000 C CNN
-F 1 "OpnTec_Logo" H 5560 4315 60  0000 C CNN
-F 2 "Custom_Components:OpnTec_Logo" H 5560 4195 60  0001 C CNN
-F 3 "" H 5560 4195 60  0001 C CNN
-	1    5560 4195
+P 5080 4195
+F 0 "S5" H 5080 4075 60  0000 C CNN
+F 1 "OpnTec_Logo" H 5080 4315 60  0000 C CNN
+F 2 "Custom_Components:OpnTec_Logo" H 5080 4195 60  0001 C CNN
+F 3 "" H 5080 4195 60  0001 C CNN
+	1    5080 4195
 	1    0    0    -1
 $EndComp
@@
 L PSLab:Logos S10
 U 1 1 5C27CF8C
-P 6460 4195
-F 0 "S10" H 6460 4075 60  0000 C CNN
-F 1 "FOSSASIA_Logo_L" H 6460 4315 60  0000 C CNN
-F 2 "Custom_Components:FOSSASIA_LogoL" H 6460 4195 60  0001 C CNN
-F 3 "" H 6460 4195 60  0001 C CNN
-	1    6460 4195
+P 5980 4195
+F 0 "S10" H 5980 4075 60  0000 C CNN
+F 1 "FOSSASIA_Logo_L" H 5980 4315 60  0000 C CNN
+F 2 "Custom_Components:FOSSASIA_LogoL" H 5980 4195 60  0001 C CNN
+F 3 "" H 5980 4195 60  0001 C CNN
+	1    5980 4195
 	1    0    0    -1
 $EndComp
+$Comp
+L PSLab:Logos S4
+U 1 1 5CB69B79
+P 6920 4185
+F 0 "S4" H 6920 4065 60  0000 C CNN
+F 1 "PSLabDotIO_B" H 6920 4305 60  0000 C CNN
+F 2 "Custom_Components:PSLabDotIO4000" H 6920 4185 60  0001 C CNN
+F 3 "" H 6920 4185 60  0001 C CNN
+	1    6920 4185
+	1    0    0    -1
+$EndComp
