File: schematics/PSLab.sch (KiCad schematic (older format))
At the start: 79 parts, among them J1 DoublePins, J10 External Power, J3 Bluetooth, J4 I2C, J5 I2C, J6 ESP01, J7 UART/ESP, J9 SPI, Q2 MMBT3904, Q3 MMBT3906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

Commit message: refactoring schematic and updated 3D parts
Parts:
- added C45: 2.2uF, Capacitor_SMD:C_0603_1608Metric, symbol Device:C
- added C46: 10uF, Capacitor_SMD:C_0603_1608Metric, symbol Device:C
- added C47: 100uF, Capacitors_Tantalum_SMD:CP_Tantalum_Case-C_EIA-6032-28_Reflow, symbol Device:C
- added J11: Battery Connector, Connector_PinSocket_2.54mm:PinSocket_1x02_P2.54mm_Vertical, symbol Connector_Generic:Conn_01x02
- added L2: 2.2uH, Inductor_SMD:L_Coilcraft_XAL5030, symbol Device:L
- added Q4: Q_NMOS_DGS, symbol Device:Q_NMOS_DGS
- added R61: 2K, Resistor_SMD:R_0603_1608Metric, symbol Device:R
- added R62: 6m, Resistor_SMD:R_0603_1608Metric, symbol Device:R
- added R63, R65, R67: 1690K, Resistor_SMD:R_0603_1608Metric, symbol Device:R
- added R64, R66, R68: 324K, Resistor_SMD:R_0603_1608Metric, symbol Device:R
- added U18: LTC4040, PSLab:LTC4040, symbol PSLab:LTC4040
- MH1: footprint Mounting_Holes:MountingHole_3.2mm_M3_DIN965_Pad -> MountingHole:MountingHole_3.2mm_M3_DIN965_Pad; symbol PSLab-rescue:CONN_1 -> Mechanical:MountingHole_Pad
- MH2, MH3, MH4: symbol PSLab-rescue:CONN_1 -> Mechanical:MountingHole_Pad
Connections:
- net labels added: BATT, IGATE, NTC, PFI, VINPUT, VSYS
- wire segments 283 -> 359
- no-connect marks 12 -> 17
Other:
- note added: "Battery Backup System"

Commit message: refactor: removed separate sch for SD Card
Parts:
- added P1: SDCard, PSLab:microSD_HC_Hirose_DM3AT-SF-PEJM5, symbol PSLab:SDCard
- added Z10: ESD-Logo, Symbol:ESD-Logo_6.6x6mm_SilkScreen, symbol PSLab:Logos
- added Z11: OpenHardware, Symbol:OSHW-Logo_5.7x6mm_SilkScreen, symbol PSLab:Logos
- added Z7: PSLab BarCode, PSLab:Barcode, symbol PSLab:Logos
- added Z8: QR Code, PSLab:Website_QR, symbol PSLab:Logos
- added Z9: BottomSilk, PSLab:PSLabRearSilk, symbol PSLab:Logos
Connections:
- no-connect marks 17 -> 21
Other:
- note added: "Logos"
Changed lines of the file:
@@
 $Descr A2 23386 16535
 encoding utf-8
-Sheet 1 6
+Sheet 1 4
 Title "PSLab Board Schematic"
 Date "2021-03-28"
@@
 Text GLabel 6775 1895 1    47   Input ~ 0
 Vdd
-$Sheet
-S 5670 5355 705  360
-U 5C27B0EA
-F0 "Logos" 61
-F1 "Logos.sch" 61
-$EndSheet
 Text GLabel 5350 2300 1    47   Input ~ 0
 SDI
@@
 NoConn ~ 1850 6090
 NoConn ~ 1850 5990
-$Sheet
-S 6830 5300 530  450
-U 5C58AFEF
-F0 "SD" 59
-F1 "SD.sch" 59
-F2 "GND" I R 7360 5670 39
-F3 "CS" O L 6830 5380 39
-F4 "MOSI" O L 6830 5480 39
-F5 "SCK" O L 6830 5580 39
-F6 "MISO" O L 6830 5680 39
-F7 "3.3V" O R 7360 5380 39
-$EndSheet
-Text GLabel 6800 5580 0    47   Input ~ 0
+Text GLabel 19975 13450 0    47   Input ~ 0
 SCK
-Text GLabel 7410 5380 2    47   Input ~ 0
+Text GLabel 19975 13350 0    47   Input ~ 0
 Vdd
-$Comp
-L PSLab-rescue:GND-RESCUE-proto1 #PWR052
-U 1 1 5C572B91
-P 7470 5740
-F 0 "#PWR052" H 7470 5740 30  0001 C CNN
-F 1 "GND" H 7470 5670 30  0001 C CNN
-F 2 "" H 7470 5740 60  0000 C CNN
-F 3 "" H 7470 5740 60  0000 C CNN
-	1    7470 5740
-	1    0    0    -1
-$EndComp
-Wire Wire Line
-	7470 5740 7470 5670
-Wire Wire Line
-	7470 5670 7360 5670
-Wire Wire Line
-	7360 5380 7410 5380
-Wire Wire Line
-	6830 5580 6800 5580
 Text GLabel 3650 3400 0    47   Input ~ 0
 CS.CH3
-Text GLabel 6810 5380 0    47   Input ~ 0
+Text GLabel 19975 13150 0    47   Input ~ 0
 CS.CH3
-Wire Wire Line
-	6810 5380 6830 5380
-Text GLabel 6800 5480 0    47   Input ~ 0
+Text GLabel 19975 13250 0    47   Input ~ 0
 SDO
-Wire Wire Line
-	6800 5480 6830 5480
-Text GLabel 6790 5680 0    47   Input ~ 0
+Text GLabel 19975 13650 0    47   Input ~ 0
 SDI
-Wire Wire Line
-	6830 5680 6790 5680
 $Comp
 L power:PWR_FLAG #FLG053
@@
 Text Notes 17125 15050 0    40   ~ 8
 Mounting Holes
+$Comp
+L PSLab:Logos Z?
+U 1 1 60674244
+P 17600 14600
+AR Path="/5C27B0EA/60674244" Ref="Z?"  Part="1"
+AR Path="/60674244" Ref="Z11"  Part="1"
+F 0 "Z11" H 17600 14480 39  0000 C CNN
+F 1 "OpenHardware" H 17600 14720 39  0000 C CNN
+F 2 "Symbol:OSHW-Logo_5.7x6mm_SilkScreen" H 17600 14600 60  0001 C CNN
+F 3 "" H 17600 14600 60  0001 C CNN
+	1    17600 14600
+	-1   0    0    1
+$EndComp
+$Comp
+L PSLab:Logos Z?
+U 1 1 6067424A
+P 17600 14200
+AR Path="/5C27B0EA/6067424A" Ref="Z?"  Part="1"
+AR Path="/6067424A" Ref="Z10"  Part="1"
+F 0 "Z10" H 17600 14080 39  0000 C CNN
+F 1 "ESD-Logo" H 17600 14320 39  0000 C CNN
+F 2 "Symbol:ESD-Logo_6.6x6mm_SilkScreen" H 17600 14200 60  0001 C CNN
+F 3 "" H 17600 14200 60  0001 C CNN
+	1    17600 14200
+	-1   0    0    1
+$EndComp
+$Comp
+L PSLab:Logos Z?
+U 1 1 60674250
+P 17600 13000
+AR Path="/5C27B0EA/60674250" Ref="Z?"  Part="1"
+AR Path="/60674250" Ref="Z7"  Part="1"
+F 0 "Z7" H 17600 12880 39  0000 C CNN
+F 1 "PSLab BarCode" H 17600 13120 39  0000 C CNN
+F 2 "PSLab:Barcode" H 17600 13000 60  0001 C CNN
+F 3 "" H 17600 13000 60  0001 C CNN
+	1    17600 13000
+	-1   0    0    1
+$EndComp
+$Comp
+L PSLab:Logos Z?
+U 1 1 60674256
+P 17600 13400
+AR Path="/5C27B0EA/60674256" Ref="Z?"  Part="1"
+AR Path="/60674256" Ref="Z8"  Part="1"
+F 0 "Z8" H 17600 13280 39  0000 C CNN
+F 1 "QR Code" H 17600 13520 39  0000 C CNN
+F 2 "PSLab:Website_QR" H 17600 13400 60  0001 C CNN
+F 3 "" H 17600 13400 60  0001 C CNN
+	1    17600 13400
+	-1   0    0    1
+$EndComp
+$Comp
+L PSLab:Logos Z?
+U 1 1 6067425C
+P 17600 13800
+AR Path="/5C27B0EA/6067425C" Ref="Z?"  Part="1"
+AR Path="/6067425C" Ref="Z9"  Part="1"
+F 0 "Z9" H 17600 13680 39  0000 C CNN
+F 1 "BottomSilk" H 17600 13920 39  0000 C CNN
+F 2 "PSLab:PSLabRearSilk" H 17600 13800 60  0001 C CNN
+F 3 "" H 17600 13800 60  0001 C CNN
+	1    17600 13800
+	-1   0    0    1
+$EndComp
 Wire Notes Line
-	17100 15775 18075 15775
+	18075 14825 17100 14825
 Wire Notes Line
-	18075 15775 18075 14950
+	17100 14825 17100 12700
+Wire Notes Line
+	17100 12700 18075 12700
+Wire Notes Line
+	18075 12700 18075 14825
 Wire Notes Line
 	18075 14950 17100 14950
 Wire Notes Line
+	18075 15775 18075 14950
+Wire Notes Line
+	17100 15775 18075 15775
+Wire Notes Line
 	17100 14950 17100 15775
+Text Notes 17125 12800 0    40   ~ 8
+Logos
+$Comp
+L PSLab:SDCard P?
+U 1 1 60642567
+P 20525 13200
+AR Path="/5C58AFEF/60642567" Ref="P?"  Part="1"
+AR Path="/60642567" Ref="P1"  Part="1"
+F 0 "P1" H 20525 12450 47  0000 C CNN
+F 1 "SDCard" H 20525 13450 47  0000 C CNN
+F 2 "PSLab:microSD_HC_Hirose_DM3AT-SF-PEJM5" H 20525 13200 60  0001 C CNN
+F 3 "https://eu.mouser.com/datasheet/2/185/DM3_catalog-939223.pdf" H 20525 13200 60  0001 C CNN
+F 4 "8P R/A SMT MICRO SD PUSH-PUSH" H 20525 13200 50  0001 C CNN "Description"
+F 5 "DM3AT-SF-PEJM5(11)" H 20525 13200 50  0001 C CNN "Mfr No."
+F 6 "DM3AT-SF-PEJM5(11)" H 20525 13200 50  0001 C CNN "PartNumber"
+F 7 "2.45" H 20525 13200 50  0001 C CNN "Price"
+	1    20525 13200
+	1    0    0    -1
+$EndComp
+NoConn ~ 19975 13050
+NoConn ~ 19975 13750
+NoConn ~ 19975 13850
+NoConn ~ 21025 13400
+$Comp
+L PSLab-rescue:GND-RESCUE-proto1 #PWR052
+U 1 1 606BCCD4
+P 20525 14125
+F 0 "#PWR052" H 20525 14125 30  0001 C CNN
+F 1 "GND" H 20525 14055 30  0001 C CNN
+F 2 "" H 20525 14125 60  0000 C CNN
+F 3 "" H 20525 14125 60  0000 C CNN
+	1    20525 14125
+	1    0    0    -1
+$EndComp
+Wire Wire Line
+	21025 13500 21275 13500
+Wire Wire Line
+	21275 13500 21275 14075
+Wire Wire Line
+	21275 14075 20525 14075
+Wire Wire Line
+	19700 14075 19700 13550
+Wire Wire Line
+	19700 13550 19975 13550
+Wire Wire Line
+	20525 14125 20525 14075
+Connection ~ 20525 14075
+Wire Wire Line
+	20525 14075 19700 14075
 $EndSCHEMATC

Commit message: refactor: rearranging USB C port sch
Parts:
- added R59, R60: 5K1, Resistor_SMD:R_0603_1608Metric, symbol Device:R
- added SW3: USB_C - Generic, Connector_USB:USB_C_Receptacle_XKB_U262-16XN-4BVC11, symbol PSLab:USB_C_Receptacle
- D6: value D -> LL4148
Connections:
- net labels added: VUSBIN
- wire segments 359 -> 376
- no-connect marks 21 -> 23
Other:
- moved on the sheet: D5, D6, Z3, Z4, Z5

Commit message: refactor: moved circuit protection to main sch
Parts:
- removed R67: 1690K, Resistor_SMD:R_0603_1608Metric, symbol Device:R
- removed R68: 324K, Resistor_SMD:R_0603_1608Metric, symbol Device:R
- added U16: SP0503BAHT, Package_TO_SOT_SMD:SOT-143, symbol Power_Protection:SP0503BAHT
- F1: value 0.5A -> 1A; symbol Device:Fuse -> Device:Polyfuse
- J11: value Battery Connector -> Li-Ion Battery
- R65: value 1690K -> 178K
- R66: value 324K -> 60.4K
- Z3: value Vbus -> VBUS
Connections:
- net labels added: CC1, CC2, CLN, L_SW
- wire segments 376 -> 363
Other:
- note added: "Circuit Protection"
- note added: "USB Connection\nTest Points BCu."
- note added: "USB Port"
- note added: "tssop-14"
- moved on the sheet: C45, C46, C47, J11, L2, Q4, R59, R60, R61, R62, R63, R64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

Commit message: refactor: removed 5V regulator
Parts:
- removed C3: 10u, Capacitor_SMD:C_0603_1608Metric, symbol Device:C
- removed C5: 1u, Capacitor_SMD:C_0603_1608Metric, symbol Device:C
- removed F2: 1.5A, Fuse:Fuse_1206_3216Metric, symbol Device:Fuse
- removed J10: External Power, Connector_PinSocket_2.54mm:PinSocket_1x03_P2.54mm_Vertical, symbol Connector_Generic:Conn_01x03
- removed SW1: Power Route, Button_Switch_THT:SW_CuK_JS202011CQN_DPDT_Straight, symbol Switch:SW_Push_DPDT
- removed U17: LDL212PU50R, Package_DFN_QFN:DFN-6-1EP_3x3mm_P0.95mm_EP1.7x2.6mm, symbol PSLab:LDL212PU50R
Connections:
- net labels removed: ExP, InP
- wire segments 363 -> 340
- no-connect marks 23 -> 22
Other:
- note removed: "External Power"
Changed lines of the file:
@@
 	2475 3750 2350 3750
 Wire Wire Line
-	2475 3210 2475 3350
+	2475 3210 2475 3225
 Wire Wire Line
 	2350 3450 2475 3450
@@
 	1    0    0    -1
 $EndComp
-$Comp
-L PSLab-rescue:GND-RESCUE-proto1 #PWR0101
-U 1 1 5EF48D55
-P 10155 830
-F 0 "#PWR0101" H 10155 830 30  0001 C CNN
-F 1 "GND" H 10155 760 30  0001 C CNN
-F 2 "" H 10155 830 60  0000 C CNN
-F 3 "" H 10155 830 60  0000 C CNN
-	1    10155 830
-	0    -1   -1   0
-$EndComp
-Wire Wire Line
-	10155 830  10100 830
 Wire Notes Line
 	3250 5585 3250 6680
 Wire Notes Line
 	535  6680 5490 6680
-$Comp
-L Device:C C3
-U 1 1 5F084CC5
-P 9845 1825
-F 0 "C3" H 9710 1930 39  0000 L CNN
-F 1 "10u" H 9715 1715 39  0000 L CNN
-F 2 "Capacitor_SMD:C_0603_1608Metric" H 9883 1675 50  0001 C CNN
-F 3 "https://eu.mouser.com/datasheet/2/396/mlcc02_e-1307760.pdf" H 9845 1825 50  0001 C CNN
-F 4 "16V 20%" H 9845 1825 50  0001 C CNN "Description"
-F 5 "EMK107BC6106MA-T" H 9845 1825 50  0001 C CNN "Mfr No."
-F 6 "0.46" H 9845 1825 50  0001 C CNN "Price"
-F 7 "EMK107BC6106MA-T" H 9845 1825 50  0001 C CNN "PartNumber"
-	1    9845 1825
-	1    0    0    -1
-$EndComp
 Wire Notes Line
 	8040 550  8040 2175
 Wire Notes Line
 	9510 2175 9510 550
-$Comp
-L Device:C C5
-U 1 1 5F12BFF6
-P 10945 1825
-F 0 "C5" H 11000 1935 39  0000 L CNN
-F 1 "1u" H 11005 1720 39  0000 L CNN
-F 2 "Capacitor_SMD:C_0603_1608Metric" H 10983 1675 50  0001 C CNN
-F 3 "https://eu.mouser.com/datasheet/2/40/cx5r-776519.pdf" H 10945 1825 50  0001 C CNN
-F 4 "16V 20%" H 10945 1825 50  0001 C CNN "Description"
-F 5 "0603YD105KAT2A" H 10945 1825 50  0001 C CNN "Mfr No."
-F 6 "0.18" H 10945 1825 50  0001 C CNN "Price"
-F 7 "0603YD105KAT2A" H 10945 1825 50  0001 C CNN "PartNumber"
-	1    10945 1825
-	1    0    0    -1
-$EndComp
-$Comp
-L PSLab-rescue:GND-RESCUE-proto1 #PWR0102
-U 1 1 5F12D03B
-P 10945 2065
-F 0 "#PWR0102" H 10945 2065 30  0001 C CNN
-F 1 "GND" H 10945 1995 30  0001 C CNN
-F 2 "" H 10945 2065 60  0000 C CNN
-F 3 "" H 10945 2065 60  0000 C CNN
-	1    10945 2065
-	1    0    0    -1
-$EndComp
-$Comp
-L PSLab-rescue:GND-RESCUE-proto1 #PWR0103
-U 1 1 5F12E11F
-P 9845 2065
-F 0 "#PWR0103" H 9845 2065 30  0001 C CNN
-F 1 "GND" H 9845 1995 30  0001 C CNN
-F 2 "" H 9845 2065 60  0000 C CNN
-F 3 "" H 9845 2065 60  0000 C CNN
-	1    9845 2065
-	1    0    0    -1
-$EndComp
-Text GLabel 9795 1520 0    39   Input ~ 8
-ExP
-$Comp
-L Connector_Generic:Conn_01x03 J10
-U 1 1 5EF478E2
-P 9900 930
-F 0 "J10" H 9818 629 39  0000 C CNN
-F 1 "External Power" H 9830 715 39  0000 C CNN
-F 2 "Connector_PinSocket_2.54mm:PinSocket_1x03_P2.54mm_Vertical" H 9900 930 50  0001 C CNN
-F 3 "https://eu.mouser.com/datasheet/2/527/ssw_th-1507658.pdf" H 9900 930 50  0001 C CNN
-F 4 "Straight female 2.54 mm 1row" H 9900 930 50  0001 C CNN "Description"
-F 5 "SSW-103-01-T-S" H 9900 930 50  0001 C CNN "Mfr No."
-F 6 "0.5" H 9900 930 50  0001 C CNN "Price"
-F 7 "SSW-103-01-T-S" H 9900 930 50  0001 C CNN "PartNumber"
-	1    9900 930
-	-1   0    0    1
-$EndComp
-$Comp
-L Device:Fuse F2
-U 1 1 5F2A4A6D
-P 10690 930
-F 0 "F2" V 10517 930 39  0000 C CNN
-F 1 "1.5A" V 10592 930 39  0000 C CNN
-F 2 "Fuse:Fuse_1206_3216Metric" V 10620 930 50  0001 C CNN
-F 3 "https://www.mouser.fi/datasheet/2/240/Littelfuse_PTC_1812L_Datasheet.pdf-693388.pdf" H 10690 930 50  0001 C CNN
-F 4 "Hold 1A, Trip 1.8A" H 10690 930 50  0001 C CNN "Description"
-F 5 "0ZCJ0100FF2E" H 10690 930 50  0001 C CNN "Mfr No."
-F 6 "0.17" H 10690 930 50  0001 C CNN "Price"
-F 7 "0ZCJ0100FF2E" H 10690 930 50  0001 C CNN "PartNumber"
-	1    10690 930
-	0    1    1    0
-$EndComp
-Wire Wire Line
-	10840 930  10945 930
-Wire Wire Line
-	10540 930  10100 930
-$Comp
-L power:PWR_FLAG #FLG0104
-U 1 1 5F320ECD
-P 3710 6550
-F 0 "#FLG0104" H 3710 6645 30  0001 C CNN
-F 1 "PWR_FLAG" V 3710 6785 30  0000 C CNN
-F 2 "" H 3710 6550 60  0000 C CNN
-F 3 "" H 3710 6550 60  0000 C CNN
-	1    3710 6550
-	0    1    1    0
-$EndComp
-$Comp
-L PSLab:LDL212PU50R U17
-U 1 1 5EF1AD6F
-P 10390 1420
-F 0 "U17" H 10390 1736 39  0000 C CNN
-F 1 "LDL212PU50R" H 10390 1661 39  0000 C CNN
-F 2 "Package_DFN_QFN:DFN-6-1EP_3x3mm_P0.95mm_EP1.7x2.6mm" H 10390 1420 39  0001 C CNN
-F 3 "https://eu.mouser.com/datasheet/2/389/dm00225720-1798688.pdf" H 10390 1420 39  0001 C CNN
-F 4 "DFN-6-1EP_3x3mm_Pitch0.95mm" H 10390 1420 50  0001 C CNN "Description"
-F 5 "LDL212PU50R" H 10390 1420 50  0001 C CNN "Mfr No."
-F 6 "LDL212PU50R" H 10390 1420 50  0001 C CNN "PartNumber"
-F 7 "0.51" H 10390 1420 50  0001 C CNN "Price"
-	1    10390 1420
-	1    0    0    -1
-$EndComp
-$Comp
-L power:PWR_FLAG #FLG0103
-U 1 1 5F31B7ED
-P 9845 1490
-F 0 "#FLG0103" H 9845 1585 30  0001 C CNN
-F 1 "PWR_FLAG" H 9845 1625 30  0000 C CNN
-F 2 "" H 9845 1490 60  0000 C CNN
-F 3 "" H 9845 1490 60  0000 C CNN
-	1    9845 1490
-	1    0    0    -1
-$EndComp
-NoConn ~ 10740 1420
-Wire Wire Line
-	9845 2065 9845 2020
-Wire Wire Line
-	9845 2020 9605 2020
-Wire Wire Line
-	9605 2020 9605 1320
-Wire Wire Line
-	9605 1320 10040 1320
-Connection ~ 9845 2020
-Wire Wire Line
-	9845 2020 9845 1975
-Wire Wire Line
-	10040 1420 9985 1420
-Wire Wire Line
-	9985 1420 9985 1520
-Wire Wire Line
-	9985 1520 10040 1520
-Wire Wire Line
-	10740 1520 10945 1520
-Wire Wire Line
-	10740 1320 10945 1320
-Wire Wire Line
-	10945 1320 10945 1520
-Connection ~ 10945 1520
-Wire Wire Line
-	10945 1520 10945 1675
-Wire Wire Line
-	10945 930  10945 1320
-Connection ~ 10945 1320
-Wire Wire Line
-	9845 1490 9845 1520
-Wire Wire Line
-	9845 1520 9795 1520
-Wire Wire Line
-	9845 1520 9985 1520
-Connection ~ 9845 1520
-Connection ~ 9985 1520
-Wire Wire Line
-	9845 1520 9845 1675
 Wire Notes Line
 	11130 550  11130 2175
@@
 Wire Notes Line
 	8040 550  11130 550
-Text Notes 10420 655  0    60   ~ 0
-External Power
 Text GLabel 2975 5990 2    39   Input ~ 8
 +5V
@@
 	2975 5990 2945 5990
 Connection ~ 2945 5990
-Wire Wire Line
-	10945 1975 10945 2020
-Wire Wire Line
-	10465 2020 10945 2020
-Wire Wire Line
-	10465 1695 10465 2020
-Connection ~ 10945 2020
-Wire Wire Line
-	10945 2020 10945 2065
 Wire Notes Line
 	7750 2270 11150 2270
@@
 	0    1    1    0
 $EndComp
-$Comp
-L Switch:SW_Push_DPDT SW1
-U 1 1 5EF8C80A
-P 3745 6070
-F 0 "SW1" H 3560 6395 39  0000 C CNN
-F 1 "Power Route" H 3900 6475 39  0000 C CNN
-F 2 "Button_Switch_THT:SW_CuK_JS202011CQN_DPDT_Straight" H 3745 6270 50  0001 C CNN
-F 3 "https://eu.mouser.com/datasheet/2/60/js-1841892.pdf" H 3745 6270 50  0001 C CNN
-F 4 "JS202011CQN" H 3745 6070 50  0001 C CNN "Mfr No."
-F 5 "JS202011CQN" H 3745 6070 50  0001 C CNN "PartNumber"
-F 6 "Slide Switches DPDT THRU HOLE" H 3745 6070 50  0001 C CNN "Description"
-F 7 "0.43" H 3745 6070 50  0001 C CNN "Price"
-	1    3745 6070
-	1    0    0    -1
-$EndComp
-Text GLabel 3945 5770 2    39   Input ~ 8
-InP
-Text GLabel 3945 6170 2    39   Input ~ 8
-InP
-Text GLabel 3945 5970 2    39   Input ~ 8
-ExP
-Text GLabel 3945 6370 2    39   Input ~ 8
-ExP
-Text GLabel 3545 6270 0    39   Input ~ 8
-+5V
-Text GLabel 3545 5870 0    39   Input ~ 8
-+5V
 Wire Notes Line
 	4165 5585 4165 6680
 Wire Notes Line
 	535  5585 4165 5585
-Text GLabel 3710 6550 0    39   Input ~ 8
-+5V
 $Comp
 L PSLab:Logos TP5
@@
 Text GLabel 7175 1895 1    47   Input ~ 0
 IOut
-Text GLabel 10100 1030 2    40   Input ~ 0
-+5V
 $Comp
 L Device:D_Zener_Small_ALT D1
@@
 Text Label -4950 5325 0    39   ~ 0
 CLN
+$Comp
+L power:PWR_FLAG #FLG?
+U 1 1 606BAE10
+P 2475 3225
+AR Path="/5ED254D7/606BAE10" Ref="#FLG?"  Part="1"
+AR Path="/606BAE10" Ref="#FLG0103"  Part="1"
+F 0 "#FLG0103" H 2475 3300 50  0001 C CNN
+F 1 "PWR_FLAG" H 2475 3398 39  0001 C CNN
+F 2 "" H 2475 3225 50  0001 C CNN
+F 3 "~" H 2475 3225 50  0001 C CNN
+	1    2475 3225
+	0    -1   -1   0
+$EndComp
+Connection ~ 2475 3225
+Wire Wire Line
+	2475 3225 2475 3350
 $EndSCHEMATC

Commit message: refactor: moved separate UART sch to main
Parts:
- added C43: 0.1uF, Capacitor_SMD:C_0603_1608Metric, symbol PSLab-rescue:C_Small
- added C44: 10uF, Capacitor_SMD:C_0603_1608Metric, symbol PSLab-rescue:C_Small
- added R48: 5K1, Resistor_SMD:R_0603_1608Metric, symbol PSLab-rescue:R
- added R51: 1K, Resistor_SMD:R_0603_1608Metric, symbol PSLab-rescue:R
- added R58: 10K, Resistor_SMD:R_0603_1608Metric, symbol PSLab-rescue:R
- added U15: CP2102N, Package_DFN_QFN:QFN-24-1EP_4x4mm_P0.5mm_EP2.6x2.6mm, symbol PSLab:CP2102
- J11: footprint Connector_PinSocket_2.54mm:PinSocket_1x02_P2.54mm_Vertical -> Connector_JST:JST_EH_S2B-EH_1x02_P2.50mm_Horizontal
- R54, R55: symbol PSLab-rescue:R-RESCUE-proto1 -> Device:R
- TP4: value TEST -> GND
Connections:
- net VSYS is gone; now on net +5V: C47.1, Q4.1 (D), R63.1, U18.1 (VSYS), U18.12 (F2), U18.13 (F1), U18.14 (F0), U18.24 (VSYS)
- net +5V: now also R48.1
- net D+: now also U15.3 (D+)
- net D-: now also U15.4 (D-)
- net GND: now also C43.2, C44.2, R58.1, U15.2 (GND), U15.25 (GND)
- net MRxD: now also U15.20 (RXD)
- net MTxD: now also U15.21 (TXD)
- net Vdd renamed +3V3
- net +3V3: now also C43.1, C44.1, R51.2, U15.5 (VIO), U15.6 (VDD), U15.7 (VREGIN)
- new net UARTReset: R51.1, U15.9 (RSTb)
- new net VBusSense: R48.2, R58.2, U15.8 (VBUS)
- no-connect marks 22 -> 36
Other:
- note added: "USB to UART Bridge"
- note removed: "USB & Power Connector , USB-UART Convertor"
- moved on the sheet: C45, C46, C47, F1, J11, L2, Q4, R54, R55, R59, R60, R61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

Commit message: refactor: removed ESP UART resistors
Parts:
- removed R56, R57: 18, Resistor_SMD:R_0603_1608Metric, symbol PSLab-rescue:R-RESCUE-proto1
- added U17: TC7662Bx0A, Package_SO:SOIC-8_3.9x4.9mm_P1.27mm, symbol Converter_DCDC:TC7662Bx0A
- C47: footprint Capacitors_Tantalum_SMD:CP_Tantalum_Case-C_EIA-6032-28_Reflow -> Capacitor_Tantalum_SMD:CP_EIA-6032-28_Kemet-C
- J11: footprint Connector_JST:JST_EH_S2B-EH_1x02_P2.50mm_Horizontal -> Connector_JST:JST_EH_B2B-EH-A_1x02_P2.50mm_Vertical
- Q2: symbol PSLab-rescue:MMBT3904 -> Transistor_BJT:MMBT3904
- Q3: symbol PSLab-rescue:MMBT3906 -> Transistor_BJT:MMBT3906
Connections:
- net ERxD is gone; now on net PGC2: J6.2 (TX)
- net ETxD is gone; now on net PGD2: J6.7 (RX)
- net AVdd renamed VDDA
Other:
- moved on the sheet: C10, C11, C12, C13, C14, C15, C16, C17, C18, C19, C2, C20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
