File: schematics/PSLab.kicad_sch (KiCad schematic)
At the start: 195 parts, among them J1 DoublePins, J10 Programmer, J11 Battery_Cell, J12 USB_C - Generic, J13 CR1225, J2 Conn_01x25, J3 Conn_01x13, J6 ESP01, J8 Micro_SD_Card_Det_9_pin, Q1 MMBT3906, Q2 MMBT3904, Q3 MMBT3906, SW1 SW_MEC_5E, SW2 SW_MEC_5E, SW3 SW_MEC_5E, U1 AP3015A, U10 TL082, U11 TL082, U12 74HC4051, U13 TL082, U14 MCP6S21-I/SN, U15 CP2102N-xxx-xQFN20x, U16 SP0503BAHT, U17 MT1470, U18 MCP6S21-I/SN, U2 74HC126, U20 MCP4822, U21 IP5189T, U3 PIC24EP256GP204, U4 DS1307Z+T&R, U6 AMS1117-3.3, U7 LM324, U9 TL082, X1 12MHz, X2 32.768 kHz

Commit message: fix: resolved all erc issues in schematic
Parts:
- D3, D4: symbol Device:LED_ALT -> Device:LED_Filled
- J12: value USB_C - Generic -> USB_C_Receptacle
- U14, U18: value MCP6S21-I/SN -> MCP6S21
Connections:
- net +3V3 is gone; now on net +3.3V: C13.1, C15.2, C4.1, J10.2 (Pin_2), J2.13 (Pin_13), J2.6 (Pin_6), J2.9 (Pin_9), J8.4 (VDD), L1.2, R1.1, R2.2, R3.2, R64.2, R66.2, R67.2, R71.2, R72.2, R73.2, U12.16 (VCC), U3.28 (VDD), U3.40 (VDD), U6.2 (VO)
- no-connect marks 34 -> 32

Commit message: chore: reduce brightness of charging LED by adding resistors
Parts:
- added R13, R27, R28, R62: 200, Resistor_SMD:R_0603_1608Metric, symbol Device:R_Small
Connections:
- net LD1: now also R28.2, R62.2; no longer D12.2 (A), D13.1 (K)
- net LD2: now also R13.2, R27.2; no longer D10.2 (A), D11.1 (K)
- new net: D11.1 (K), R27.1
- new net: D10.2 (A), R13.1
- new net: D13.1 (K), R62.1
- new net: D12.2 (A), R28.1

Commit message: chore: move socket inner, change pin to socket
Parts:
- J2: footprint Connector_PinHeader_2.54mm:PinHeader_1x25_P2.54mm_Vertical -> Connector_PinSocket_2.54mm:PinSocket_1x25_P2.54mm_Vertical
- J3: footprint Connector_PinHeader_2.54mm:PinHeader_1x13_P2.54mm_Vertical -> Connector_PinSocket_2.54mm:PinSocket_1x13_P2.54mm_Vertical
Changed lines of the file:
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@@
       (effects (font (size 1.27 1.27)))
     )
-    (property "Footprint" "Connector_PinHeader_2.54mm:PinHeader_1x25_P2.54mm_Vertical" (at 373.38 236.22 0)
+    (property "Footprint" "Connector_PinSocket_2.54mm:PinSocket_1x25_P2.54mm_Vertical" (at 373.38 236.22 0)
       (effects (font (size 1.27 1.27)) hide)
     )
@@
       (effects (font (size 1.27 1.27)))
     )
-    (property "Footprint" "Connector_PinHeader_2.54mm:PinHeader_1x13_P2.54mm_Vertical" (at 441.96 236.22 0)
-      (effects (font (size 1.27 1.27)) hide)
-    )
+    (property "Footprint" "Connector_PinSocket_2.54mm:PinSocket_1x13_P2.54mm_Vertical" (at 441.96 236.22 0)
+      (effects (font (size 1.27 1.27)) hide)
+    )

Commit message: fix: resolved design rules issues and workflow
Parts:
- removed Z8: QR Code, PSLab:Website_QR, symbol PSLab:Logos
- D1, D2: symbol Device:D_Zener_Small_ALT -> Device:D_Zener_Small_Filled
- D8: symbol Diode:1N4148W -> Device:D
- D9: footprint Diode_SMD:D_MiniMELF -> Diode_SMD:D_SOD-123
- MH1, MH2, MH3: footprint MountingHole:MountingHole_3.2mm_M3_DIN965_Pad -> PSLab:OneSided_MPad
- MH4: footprint MountingHole:MountingHole_3.2mm_M3_DIN965_Pad -> PSLab:TwoSided_MPad
- Z9: footprint PSLab:Silk -> PSLab:PSLab_SilkScreen
Other:
- note added: "I_chg = 100k * 1.2V / R_chg = 0.6A"
- note removed: "I_chg=100000 * 1.2V / R_chg =0.6A"
- moved on the sheet: C1, C13, C17, C4, MH3, MH4, R10, R12, R56, R57, Z10, Z7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
